Commit message: feat: add slam toolbox and create odometry

File: src/ackermann_description/urdf/wheels.xacro (robot description, xacro)
@@ -9,4 +9,5 @@
                 <axis xyz="0.0 0.0 1"/>
                 <limit lower="-0.5" upper="0.5" effort="0.1" velocity="1.0"/>
+                <dynamics damping="0.05" friction="0.02"/>
             </xacro:if>
         </joint>
@@ -14,5 +15,5 @@
             <inertial>
                 <origin xyz="0.0 0.0 0.0" rpy="0.0 0.0 0.0"/>
-                <mass value="0.01"/>
+                <mass value="0.05"/>
                 <inertia ixx="0.0001" ixy="0.0" ixz="0.0" iyy="0.0001" iyz="0.0" izz="0.0001"/>
             </inertial>
@@ -38,10 +39,11 @@
             <child link="${prefix}_wheel"/>
             <axis xyz="0.0 0.0 1"/>
+            <dynamics damping="0.01" friction="0.005"/>
         </joint>
         <link name="${prefix}_wheel">
             <inertial>
                 <origin xyz="0.0 0.0 0.0" rpy="0.0 0.0 0.0"/>
-                <mass value="0.1"/>
-                <inertia ixx="0.001" ixy="0.0" ixz="0.0" iyy="0.001" iyz="0.0" izz="0.001"/>
+                <mass value="0.05"/>  <!-- thay vì 0.01 -->
+                <inertia ixx="0.0003" ixy="0.0" ixz="0.0" iyy="0.0003" iyz="0.0" izz="0.0003"/>
             </inertial>
             <visual>
