Commit message: feat: nav2

File: src/ackermann_description/urdf/gazebo_control.xacro (robot description, xacro)
@@ -1,43 +1,56 @@
 <?xml version="1.0"?>
 <robot xmlns:xacro="http://www.ros.org/wiki/xacro">
-  <xacro:macro name="gazebo_control">
-    <ros2_control name="GazeboSystem" type="system">
-      <hardware>
-        <plugin>gazebo_ros2_control/GazeboSystem</plugin>
-      </hardware>
-      <joint name="front_left_steer_joint">
-        <command_interface name="position"/>
-        <state_interface name="position"/>
-        <state_interface name="velocity"/>
-      </joint>
-      <joint name="front_right_steer_joint">
-        <command_interface name="position"/>
-        <state_interface name="position"/>
-        <state_interface name="velocity"/>
-      </joint>
-      <joint name="front_left_wheel_joint">
-        <state_interface name="position"/>
-        <state_interface name="velocity"/>
-      </joint>
-      <joint name="front_right_wheel_joint">
-        <state_interface name="position"/>
-        <state_interface name="velocity"/>
-      </joint>
-      <joint name="rear_left_wheel_joint">
-        <command_interface name="velocity"/>
-        <state_interface name="position"/>
-        <state_interface name="velocity"/>
-      </joint>
-      <joint name="rear_right_wheel_joint">
-        <command_interface name="velocity"/>
-        <state_interface name="position"/>
-        <state_interface name="velocity"/>
-      </joint>
-    </ros2_control>
-    <gazebo>
-    <plugin filename="libgazebo_ros2_control.so" name="gazebo_ros2_control">
-        <parameters>$(find ackermann_description)/config/controller.yaml</parameters>
-    </plugin>
-    </gazebo>
-  </xacro:macro>
+<xacro:macro name="gazebo_control">
+<ros2_control name="GazeboSystem" type="system">
+<hardware>
+<plugin>gazebo_ros2_control/GazeboSystem</plugin>
+</hardware>
+<!-- PID gain cho khop lai - THEM MOI. Truoc day khong co gain nao ca,
+     Gazebo dung gia tri mac dinh khong tune -> gay dao dong (giat qua
+     lai) khi khop tien gan vi tri dich. p/i/d ben duoi la diem khoi
+     dau hop ly, can tinh chinh thuc te theo huong dan kiem chung ben
+     duoi cau tra loi. -->
+<joint name="front_left_steer_joint">
+<command_interface name="position">
+<param name="p">15.0</param>
+<param name="i">0.0</param>
+<param name="d">0.8</param>
+</command_interface>
+<state_interface name="position"/>
+<state_interface name="velocity"/>
+</joint>
+<joint name="front_right_steer_joint">
+<command_interface name="position">
+<param name="p">15.0</param>
+<param name="i">0.0</param>
+<param name="d">0.8</param>
+</command_interface>
+<state_interface name="position"/>
+<state_interface name="velocity"/>
+</joint>
+<joint name="front_left_wheel_joint">
+<state_interface name="position"/>
+<state_interface name="velocity"/>
+</joint>
+<joint name="front_right_wheel_joint">
+<state_interface name="position"/>
+<state_interface name="velocity"/>
+</joint>
+<joint name="rear_left_wheel_joint">
+<command_interface name="velocity"/>
+<state_interface name="position"/>
+<state_interface name="velocity"/>
+</joint>
+<joint name="rear_right_wheel_joint">
+<command_interface name="velocity"/>
+<state_interface name="position"/>
+<state_interface name="velocity"/>
+</joint>
+</ros2_control>
+<gazebo>
+<plugin filename="libgazebo_ros2_control.so" name="gazebo_ros2_control">
+<parameters>$(find ackermann_description)/config/controller.yaml</parameters>
+</plugin>
+</gazebo>
+</xacro:macro>
 </robot>

File: src/ackermann_description/urdf/wheels.xacro (robot description, xacro)
@@ -8,5 +8,5 @@
             <xacro:if value="${is_steer}">
                 <axis xyz="0.0 0.0 1"/>
-                <limit lower="-0.5" upper="0.5" effort="0.1" velocity="1.0"/>
+                <limit lower="-0.436332" upper="0.436332" effort="0.1" velocity="1.0"/>
                 <dynamics damping="0.05" friction="0.02"/>
             </xacro:if>
