Commit message: modifiedcar geometry, tf tree

File: src/ackermann_description/urdf/ackermann.urdf.xacro (robot description, xacro)
@@ -2,8 +2,44 @@
 <robot xmlns:xacro="http://www.ros.org/wiki/xacro"
        name="agv_simulation">
+  <!-- Overall envelope dimensions come from the supplied drawing.
+       Wheelbase/track are retained estimates from the existing model;
+       body profile values are adjustable estimates, not measured vertices.
+       vehicle_width is the total envelope reference, not the chassis width. -->
+  <xacro:arg name="vehicle_length" default="0.4447"/>
+  <xacro:arg name="vehicle_width" default="0.362"/>
+  <xacro:arg name="wheelbase" default="0.3187"/>
+  <xacro:arg name="front_track" default="0.3118"/>
+  <xacro:arg name="rear_track" default="0.3118"/>
+  <xacro:arg name="wheel_radius" default="0.05"/>
+  <xacro:arg name="wheel_width" default="0.0408"/>
+  <xacro:arg name="steering_axis_offset" default="0.0369"/>
+  <xacro:arg name="front_body_width" default="0.238"/>
+  <xacro:arg name="middle_body_width" default="0.180"/>
+  <xacro:arg name="rear_body_width" default="0.238"/>
+  <xacro:arg name="front_body_length" default="0.100"/>
+  <xacro:arg name="middle_body_length" default="0.1447"/>
+  <xacro:arg name="rear_body_length" default="0.100"/>
+  <xacro:arg name="chamfer_length" default="0.050"/>
+  <xacro:arg name="body_height" default="0.0184"/>
   <xacro:include filename="core_macro.xacro"/>
   <xacro:include filename="laser.xacro"/>
   <xacro:include filename="gazebo_control.xacro"/>
-  <xacro:core/>
+  <xacro:core
+    vehicle_length="$(arg vehicle_length)"
+    vehicle_width="$(arg vehicle_width)"
+    wheelbase="$(arg wheelbase)"
+    front_track="$(arg front_track)"
+    rear_track="$(arg rear_track)"
+    wheel_radius="$(arg wheel_radius)"
+    wheel_width="$(arg wheel_width)"
+    steering_axis_offset="$(arg steering_axis_offset)"
+    front_body_width="$(arg front_body_width)"
+    middle_body_width="$(arg middle_body_width)"
+    rear_body_width="$(arg rear_body_width)"
+    front_body_length="$(arg front_body_length)"
+    middle_body_length="$(arg middle_body_length)"
+    rear_body_length="$(arg rear_body_length)"
+    chamfer_length="$(arg chamfer_length)"
+    body_height="$(arg body_height)"/>
   <xacro:laser/>
   <xacro:gazebo_control/>

File: src/ackermann_description/urdf/core_macro.xacro (robot description, xacro)
@@ -3,14 +3,32 @@
     <!-- Include wheel macro -->
     <xacro:include filename="wheels.xacro" />
-    <xacro:macro name="core">
-        <!-- Base link -->
+    <xacro:macro name="body_section" params="x length width height">
+        <visual>
+            <origin xyz="${x} 0 0"/>
+            <geometry><box size="${length} ${width} ${height}"/></geometry>
+            <material name="body_material"><color rgba="0.82 0.82 0.82 1.0"/></material>
+        </visual>
+        <collision>
+            <origin xyz="${x} 0 0"/>
+            <geometry><box size="${length} ${width} ${height}"/></geometry>
+        </collision>
+    </xacro:macro>
+    <xacro:macro name="core" params="vehicle_length vehicle_width wheelbase front_track rear_track wheel_radius wheel_width steering_axis_offset front_body_width middle_body_width rear_body_width front_body_length middle_body_length rear_body_length chamfer_length body_height">
+        <!-- base_footprint is the rear-axle ground reference (x=0). -->
+        <link name="base_footprint"/>
+        <joint name="base_footprint_to_base_link_joint" type="fixed">
+            <origin xyz="${wheelbase / 2.0} 0 ${wheel_radius}" rpy="0.0 0.0 0.0"/>
+            <parent link="base_footprint"/>
+            <child link="base_link"/>
+        </joint>
         <link name="base_link"/>
-        <!-- Base footprint -->
-        <joint name="base_footprint_to_base_link_joint" type="fixed">
-            <origin xyz="0.0 0.0 0.0" rpy="0.0 0.0 0.0"/>
+        <!-- Keep the legacy rear_axle link and joint names. Its XY location
+             matches base_footprint; its Z is the wheel axle height. -->
+        <joint name="base_link_to_rear_axle_joint" type="fixed">
+            <origin xyz="${-wheelbase / 2.0} 0.0 0.0" rpy="0.0 0.0 0.0"/>
             <parent link="base_link"/>
-            <child link="base_footprint"/>
+            <child link="rear_axle"/>
         </joint>
-        <link name="base_footprint" />
+        <link name="rear_axle" />
         <!-- Chassis -->
         <joint name="chassis_joint" type="fixed">
@@ -20,20 +38,15 @@
         </joint>
         <link name="chassis">
-            <visual>
-                <origin xyz="0.0 0.0 0.0"/>
-                <geometry>
-                    <box size="0.3865 0.238 0.0184"/>
-                </geometry>
-                <material name="">
-                    <color rgba="1.0 1.0 1.0 1.0"/>
-                    <texture filename=""/>
-                </material>
-            </visual>
-            <collision>
-                <origin xyz="0.0 0.0 0.0"/>
-                 <geometry>
-                    <box size="0.3865 0.238 0.0184"/>
-                </geometry>
-            </collision>
+            <!-- Profile defaults are adjustable estimates; sections abut
+                 without overlap to keep the simplified collision stable. -->
+            <xacro:body_section x="${-vehicle_length / 2.0 + rear_body_length / 2.0}" length="${rear_body_length}" width="${rear_body_width}" height="${body_height}"/>
+            <xacro:body_section x="${-vehicle_length / 2.0 + rear_body_length + chamfer_length / 6.0}" length="${chamfer_length / 3.0}" width="${(rear_body_width * 2.0 + middle_body_width) / 3.0}" height="${body_height}"/>
+            <xacro:body_section x="${-vehicle_length / 2.0 + rear_body_length + chamfer_length / 2.0}" length="${chamfer_length / 3.0}" width="${(rear_body_width + middle_body_width) / 2.0}" height="${body_height}"/>
+            <xacro:body_section x="${-vehicle_length / 2.0 + rear_body_length + 5.0 * chamfer_length / 6.0}" length="${chamfer_length / 3.0}" width="${(rear_body_width + middle_body_width * 2.0) / 3.0}" height="${body_height}"/>
+            <xacro:body_section x="${-vehicle_length / 2.0 + rear_body_length + chamfer_length + middle_body_length / 2.0}" length="${middle_body_length}" width="${middle_body_width}" height="${body_height}"/>
+            <xacro:body_section x="${vehicle_length / 2.0 - front_body_length - 5.0 * chamfer_length / 6.0}" length="${chamfer_length / 3.0}" width="${(front_body_width + middle_body_width * 2.0) / 3.0}" height="${body_height}"/>
+            <xacro:body_section x="${vehicle_length / 2.0 - front_body_length - chamfer_length / 2.0}" length="${chamfer_length / 3.0}" width="${(front_body_width + middle_body_width) / 2.0}" height="${body_height}"/>
+            <xacro:body_section x="${vehicle_length / 2.0 - front_body_length - chamfer_length / 6.0}" length="${chamfer_length / 3.0}" width="${(front_body_width * 2.0 + middle_body_width) / 3.0}" height="${body_height}"/>
+            <xacro:body_section x="${vehicle_length / 2.0 - front_body_length / 2.0}" length="${front_body_length}" width="${front_body_width}" height="${body_height}"/>
             <inertial>
                 <origin xyz="0.0 0.0 0.0" rpy="0.0 0.0 0.0"/>
@@ -42,9 +55,12 @@
             </inertial>
         </link>
-        <!-- Wheel -->
-        <xacro:wheel_unit prefix="front_left"  parent="base_link" x_pos="0.15935"  y_pos="0.119"  side_reflect="1"  is_steer="true" />
-        <xacro:wheel_unit prefix="front_right" parent="base_link" x_pos="0.15935"  y_pos="-0.119" side_reflect="-1" is_steer="true" />
-        <xacro:wheel_unit prefix="rear_left"   parent="base_link" x_pos="-0.15935" y_pos="0.119"  side_reflect="1"  is_steer="false" />
-        <xacro:wheel_unit prefix="rear_right"  parent="base_link" x_pos="-0.15935" y_pos="-0.119" side_reflect="-1" is_steer="false" />
+        <!-- Front wheels are positioned relative to the chassis-centered
+             base_link. The rear wheels are children of rear_axle, whose frame
+             is at the rear axle height and remains coincident with x=0 in
+             base_footprint. -->
+        <xacro:wheel_unit prefix="front_left"  parent="base_link" x_pos="${wheelbase / 2.0}" y_pos="${front_track / 2.0}" z_pos="0.0" side_reflect="1" is_steer="true" wheel_radius="${wheel_radius}" wheel_width="${wheel_width}" steering_axis_offset="${steering_axis_offset}" />
+        <xacro:wheel_unit prefix="front_right" parent="base_link" x_pos="${wheelbase / 2.0}" y_pos="${-front_track / 2.0}" z_pos="0.0" side_reflect="-1" is_steer="true" wheel_radius="${wheel_radius}" wheel_width="${wheel_width}" steering_axis_offset="${steering_axis_offset}" />
+        <xacro:wheel_unit prefix="rear_left"   parent="rear_axle" x_pos="0.0" y_pos="${rear_track / 2.0}" z_pos="0.0" side_reflect="1" is_steer="false" wheel_radius="${wheel_radius}" wheel_width="${wheel_width}" steering_axis_offset="${steering_axis_offset}" />
+        <xacro:wheel_unit prefix="rear_right"  parent="rear_axle" x_pos="0.0" y_pos="${-rear_track / 2.0}" z_pos="0.0" side_reflect="-1" is_steer="false" wheel_radius="${wheel_radius}" wheel_width="${wheel_width}" steering_axis_offset="${steering_axis_offset}" />
         <!-- Laser mount -->
         <joint name="base_laser_joint" type="fixed">

File: src/ackermann_description/urdf/wheels.xacro (robot description, xacro)
@@ -1,12 +1,14 @@
 <?xml version="1.0"?>
 <robot xmlns:xacro="http://www.ros.org/wiki/xacro">
-    <xacro:macro name="wheel_unit" params="prefix parent x_pos y_pos side_reflect is_steer">
+    <xacro:macro name="wheel_unit" params="prefix parent x_pos y_pos z_pos side_reflect is_steer wheel_radius wheel_width steering_axis_offset">
         <joint name="${prefix}_steer_joint" type="${'revolute' if is_steer else 'fixed'}">
             <parent link="${parent}"/>
             <child link="${prefix}_steer_link"/>
-            <origin xyz="${x_pos} ${y_pos} 0.0" rpy="0.0 0.0 0.0"/>
+            <!-- Keep the existing kingpin-to-wheel-center offset as an
+                 adjustable estimate; y_pos denotes the tire center. -->
+            <origin xyz="${x_pos} ${y_pos - side_reflect * steering_axis_offset} ${z_pos}" rpy="0.0 0.0 0.0"/>
             <xacro:if value="${is_steer}">
                 <axis xyz="0.0 0.0 1"/>
-                <limit lower="-0.436332" upper="0.436332" effort="0.1" velocity="1.0"/>
+                <limit lower="-0.261799" upper="0.261799" effort="0.1" velocity="1.0"/>
                 <dynamics damping="0.05" friction="0.02"/>
             </xacro:if>
@@ -35,5 +37,5 @@
         </link>
         <joint name="${prefix}_wheel_joint" type="continuous">
-            <origin xyz="0.0 ${side_reflect * 0.0369} 0.0" rpy="-${pi/2} 0.0 0.0"/>
+            <origin xyz="0.0 ${side_reflect * steering_axis_offset} 0.0" rpy="-${pi/2} 0.0 0.0"/>
             <parent link="${prefix}_steer_link"/>
             <child link="${prefix}_wheel"/>
@@ -50,5 +52,5 @@
                 <origin xyz="0.0 0.0 0.0" rpy="0.0 0.0 0.0"/>
                 <geometry>
-                    <cylinder radius="0.05" length="0.0408"/>
+                    <cylinder radius="${wheel_radius}" length="${wheel_width}"/>
                 </geometry>
                 <material name="red_material">
@@ -59,5 +61,5 @@
                 <origin xyz="0.0 0.0 0.0" rpy="0.0 0.0 0.0"/>
                 <geometry>
-                    <cylinder radius="0.05" length="0.0408"/>
+                    <cylinder radius="${wheel_radius}" length="${wheel_width}"/>
                 </geometry>
             </collision>
