Commit message: Sync Ackermann ROS 2 workspace for physical robot

File: src/ackermann_description/urdf/ackermann.urdf.xacro (robot description, xacro)
@@ -2,15 +2,12 @@
 <robot xmlns:xacro="http://www.ros.org/wiki/xacro"
        name="agv_simulation">
-  <!-- Overall envelope dimensions come from the supplied drawing.
-       Wheelbase/track are retained estimates from the existing model;
-       body profile values are adjustable estimates, not measured vertices.
-       vehicle_width is the total envelope reference, not the chassis width. -->
-  <xacro:arg name="vehicle_length" default="0.4447"/>
+  <xacro:arg name="vehicle_length" default="0.3865"/>
   <xacro:arg name="vehicle_width" default="0.362"/>
   <xacro:arg name="wheelbase" default="0.3187"/>
   <xacro:arg name="front_track" default="0.3118"/>
   <xacro:arg name="rear_track" default="0.3118"/>
-  <xacro:arg name="wheel_radius" default="0.05"/>
+  <xacro:arg name="wheel_radius" default="0.063"/>
   <xacro:arg name="wheel_width" default="0.0408"/>
+  <xacro:arg name="wheel_outer_overhang" default="0.0047"/>
   <xacro:arg name="steering_axis_offset" default="0.0369"/>
   <xacro:arg name="front_body_width" default="0.238"/>
@@ -18,11 +15,13 @@
   <xacro:arg name="rear_body_width" default="0.238"/>
   <xacro:arg name="front_body_length" default="0.100"/>
-  <xacro:arg name="middle_body_length" default="0.1447"/>
+  <xacro:arg name="middle_body_length" default="0.0865"/>
   <xacro:arg name="rear_body_length" default="0.100"/>
   <xacro:arg name="chamfer_length" default="0.050"/>
-  <xacro:arg name="body_height" default="0.0184"/>
+  <xacro:arg name="body_height" default="0.0444"/>
+  <xacro:arg name="lidar_x_rear_axle" default="0.240"/>
+  <xacro:arg name="lidar_height" default="0.146"/>
+  <xacro:include filename="materials.xacro"/>
   <xacro:include filename="core_macro.xacro"/>
   <xacro:include filename="laser.xacro"/>
-  <xacro:include filename="gazebo_control.xacro"/>
   <xacro:core
     vehicle_length="$(arg vehicle_length)"
@@ -33,4 +32,5 @@
     wheel_radius="$(arg wheel_radius)"
     wheel_width="$(arg wheel_width)"
+    wheel_outer_overhang="$(arg wheel_outer_overhang)"
     steering_axis_offset="$(arg steering_axis_offset)"
     front_body_width="$(arg front_body_width)"
@@ -41,6 +41,8 @@
     rear_body_length="$(arg rear_body_length)"
     chamfer_length="$(arg chamfer_length)"
-    body_height="$(arg body_height)"/>
-  <xacro:laser/>
-  <xacro:gazebo_control/>
+    body_height="$(arg body_height)"
+    lidar_x_rear_axle="$(arg lidar_x_rear_axle)"/>
+  <xacro:laser
+    lidar_height="$(arg lidar_height)"
+    wheel_radius="$(arg wheel_radius)"/>
 </robot>

File: src/ackermann_description/urdf/core_macro.xacro (robot description, xacro)
@@ -1,5 +1,4 @@
 <?xml version="1.0"?>
 <robot xmlns:xacro="http://www.ros.org/wiki/xacro">
-    <!-- Include wheel macro -->
     <xacro:include filename="wheels.xacro" />
     <xacro:macro name="body_section" params="x length width height">
@@ -7,5 +6,5 @@
             <origin xyz="${x} 0 0"/>
             <geometry><box size="${length} ${width} ${height}"/></geometry>
-            <material name="body_material"><color rgba="0.82 0.82 0.82 1.0"/></material>
+            <material name="body_material"/>
         </visual>
         <collision>
@@ -14,7 +13,13 @@
         </collision>
     </xacro:macro>
-    <xacro:macro name="core" params="vehicle_length vehicle_width wheelbase front_track rear_track wheel_radius wheel_width steering_axis_offset front_body_width middle_body_width rear_body_width front_body_length middle_body_length rear_body_length chamfer_length body_height">
-        <!-- base_footprint is the rear-axle ground reference (x=0). -->
+    <xacro:macro name="core" params="vehicle_length vehicle_width wheelbase front_track rear_track wheel_radius wheel_width wheel_outer_overhang steering_axis_offset front_body_width middle_body_width rear_body_width front_body_length middle_body_length rear_body_length chamfer_length body_height lidar_x_rear_axle">
         <link name="base_footprint"/>
+        <joint name="base_footprint_to_imu_joint" type="fixed">
+            <!-- Temporary center-of-chassis placement; adjust after measuring the installed IMU. -->
+            <origin xyz="${wheelbase / 2.0} 0.0 ${wheel_radius}" rpy="0.0 0.0 0.0"/>
+            <parent link="base_footprint"/>
+            <child link="imu_link"/>
+        </joint>
+        <link name="imu_link"/>
         <joint name="base_footprint_to_base_link_joint" type="fixed">
             <origin xyz="${wheelbase / 2.0} 0 ${wheel_radius}" rpy="0.0 0.0 0.0"/>
@@ -23,6 +28,4 @@
         </joint>
         <link name="base_link"/>
-        <!-- Keep the legacy rear_axle link and joint names. Its XY location
-             matches base_footprint; its Z is the wheel axle height. -->
         <joint name="base_link_to_rear_axle_joint" type="fixed">
             <origin xyz="${-wheelbase / 2.0} 0.0 0.0" rpy="0.0 0.0 0.0"/>
@@ -31,5 +34,4 @@
         </joint>
         <link name="rear_axle" />
-        <!-- Chassis -->
         <joint name="chassis_joint" type="fixed">
             <parent link="base_link"/>
@@ -38,6 +40,4 @@
         </joint>
         <link name="chassis">
-            <!-- Profile defaults are adjustable estimates; sections abut
-                 without overlap to keep the simplified collision stable. -->
             <xacro:body_section x="${-vehicle_length / 2.0 + rear_body_length / 2.0}" length="${rear_body_length}" width="${rear_body_width}" height="${body_height}"/>
             <xacro:body_section x="${-vehicle_length / 2.0 + rear_body_length + chamfer_length / 6.0}" length="${chamfer_length / 3.0}" width="${(rear_body_width * 2.0 + middle_body_width) / 3.0}" height="${body_height}"/>
@@ -49,21 +49,11 @@
             <xacro:body_section x="${vehicle_length / 2.0 - front_body_length - chamfer_length / 6.0}" length="${chamfer_length / 3.0}" width="${(front_body_width * 2.0 + middle_body_width) / 3.0}" height="${body_height}"/>
             <xacro:body_section x="${vehicle_length / 2.0 - front_body_length / 2.0}" length="${front_body_length}" width="${front_body_width}" height="${body_height}"/>
-            <inertial>
-                <origin xyz="0.0 0.0 0.0" rpy="0.0 0.0 0.0"/>
-                <mass value="1.0"/>
-                <inertia ixx="0.0047" ixy="0.0" ixz="0.0" iyy="0.0125" iyz="0.0" izz="0.0171"/>
-            </inertial>
         </link>
-        <!-- Front wheels are positioned relative to the chassis-centered
-             base_link. The rear wheels are children of rear_axle, whose frame
-             is at the rear axle height and remains coincident with x=0 in
-             base_footprint. -->
-        <xacro:wheel_unit prefix="front_left"  parent="base_link" x_pos="${wheelbase / 2.0}" y_pos="${front_track / 2.0}" z_pos="0.0" side_reflect="1" is_steer="true" wheel_radius="${wheel_radius}" wheel_width="${wheel_width}" steering_axis_offset="${steering_axis_offset}" />
-        <xacro:wheel_unit prefix="front_right" parent="base_link" x_pos="${wheelbase / 2.0}" y_pos="${-front_track / 2.0}" z_pos="0.0" side_reflect="-1" is_steer="true" wheel_radius="${wheel_radius}" wheel_width="${wheel_width}" steering_axis_offset="${steering_axis_offset}" />
-        <xacro:wheel_unit prefix="rear_left"   parent="rear_axle" x_pos="0.0" y_pos="${rear_track / 2.0}" z_pos="0.0" side_reflect="1" is_steer="false" wheel_radius="${wheel_radius}" wheel_width="${wheel_width}" steering_axis_offset="${steering_axis_offset}" />
-        <xacro:wheel_unit prefix="rear_right"  parent="rear_axle" x_pos="0.0" y_pos="${-rear_track / 2.0}" z_pos="0.0" side_reflect="-1" is_steer="false" wheel_radius="${wheel_radius}" wheel_width="${wheel_width}" steering_axis_offset="${steering_axis_offset}" />
-        <!-- Laser mount -->
+        <xacro:wheel_unit prefix="front_left"  parent="base_link" x_pos="${wheelbase / 2.0}" y_pos="${front_track / 2.0}" z_pos="0.0" side_reflect="1" is_steer="true" wheel_radius="${wheel_radius}" wheel_width="${wheel_width}" wheel_outer_overhang="${wheel_outer_overhang}" steering_axis_offset="${steering_axis_offset}" />
+        <xacro:wheel_unit prefix="front_right" parent="base_link" x_pos="${wheelbase / 2.0}" y_pos="${-front_track / 2.0}" z_pos="0.0" side_reflect="-1" is_steer="true" wheel_radius="${wheel_radius}" wheel_width="${wheel_width}" wheel_outer_overhang="${wheel_outer_overhang}" steering_axis_offset="${steering_axis_offset}" />
+        <xacro:wheel_unit prefix="rear_left"   parent="rear_axle" x_pos="0.0" y_pos="${rear_track / 2.0}" z_pos="0.0" side_reflect="1" is_steer="false" wheel_radius="${wheel_radius}" wheel_width="${wheel_width}" wheel_outer_overhang="${wheel_outer_overhang}" steering_axis_offset="${steering_axis_offset}" />
+        <xacro:wheel_unit prefix="rear_right"  parent="rear_axle" x_pos="0.0" y_pos="${-rear_track / 2.0}" z_pos="0.0" side_reflect="-1" is_steer="false" wheel_radius="${wheel_radius}" wheel_width="${wheel_width}" wheel_outer_overhang="${wheel_outer_overhang}" steering_axis_offset="${steering_axis_offset}" />
         <joint name="base_laser_joint" type="fixed">
-            <origin xyz="0.0 0.0 0.0" rpy="0.0 0.0 0.0"/>
+            <origin xyz="${lidar_x_rear_axle - wheelbase / 2.0} 0.0 0.0" rpy="0.0 0.0 0.0"/>
             <parent link="chassis"/>
             <child link="base_laser"/>
@@ -75,8 +65,5 @@
                     <cylinder radius="0.06" length="0.0684"/>
                 </geometry>
-                <material name="">
-                    <color rgba="1.0 1.0 1.0 1.0"/>
-                    <texture filename=""/>
-                </material>
+                <material name="sensor_mount_material"/>
             </visual>
             <collision>
@@ -86,9 +73,4 @@
                 </geometry>
             </collision>
-            <inertial>
-                <origin xyz="0.0 0.0 0.0276" rpy="0.0 0.0 0.0"/>
-                <mass value="0.2"/>
-                <inertia ixx="0.00025" ixy="0.0" ixz="0.0" iyy="0.00025" iyz="0.0" izz="0.00036"/>
-            </inertial>
         </link>
     </xacro:macro>

File: src/ackermann_description/urdf/laser.xacro (robot description, xacro)
@@ -1,10 +1,10 @@
 <?xml version="1.0"?>
 <robot xmlns:xacro="http://www.ros.org/wiki/xacro">
-  <xacro:include filename="inertial_macros.xacro"/>
-  <xacro:macro name="laser">
+  <xacro:macro name="laser" params="lidar_height wheel_radius">
     <joint name="laser_joint" type="fixed">
       <parent link="base_laser"/>
       <child link="laser_frame"/>
-      <origin xyz="0.0 0 0.0776" rpy="0 0 0"/>
+      <!-- Convert rear-axle/ground measurements to base_link coordinates. -->
+      <origin xyz="0.0 0.0 ${lidar_height - wheel_radius}" rpy="0 0 0"/>
     </joint>
     <link name="laser_frame">
@@ -13,5 +13,5 @@
           <cylinder radius="0.05" length="0.04"/>
         </geometry>
-        <material name="red"/>
+        <material name="lidar_material"/>
       </visual>
       <collision>
@@ -20,34 +20,5 @@
         </geometry>
       </collision>
-      <xacro:inertial_cylinder mass="0.1" length="0.04" radius="0.05"/>
     </link>
-    <gazebo reference="laser_frame">
-      <material>Gazebo/Red</material>
-      <sensor name="laser" type="ray">
-        <pose> 0 0 0 0 0 0 </pose>
-        <visualize>true</visualize>
-        <update_rate>10</update_rate>
-        <ray>
-          <scan>
-            <horizontal>
-              <samples>360</samples>
-              <min_angle>-3.14</min_angle>
-              <max_angle>3.14</max_angle>
-            </horizontal>
-          </scan>
-          <range>
-            <min>0.3</min>
-            <max>12</max>
-          </range>
-        </ray>
-        <plugin name="laser_controller" filename="libgazebo_ros_ray_sensor.so">
-          <ros>
-            <argument>~/out:=scan</argument>
-          </ros>
-          <output_type>sensor_msgs/LaserScan</output_type>
-          <frame_name>laser_frame</frame_name>
-        </plugin>
-      </sensor>
-    </gazebo>
   </xacro:macro>
 </robot>

File: src/ackermann_description/urdf/wheels.xacro (robot description, xacro)
@@ -1,10 +1,8 @@
 <?xml version="1.0"?>
 <robot xmlns:xacro="http://www.ros.org/wiki/xacro">
-    <xacro:macro name="wheel_unit" params="prefix parent x_pos y_pos z_pos side_reflect is_steer wheel_radius wheel_width steering_axis_offset">
+    <xacro:macro name="wheel_unit" params="prefix parent x_pos y_pos z_pos side_reflect is_steer wheel_radius wheel_width wheel_outer_overhang steering_axis_offset">
         <joint name="${prefix}_steer_joint" type="${'revolute' if is_steer else 'fixed'}">
             <parent link="${parent}"/>
             <child link="${prefix}_steer_link"/>
-            <!-- Keep the existing kingpin-to-wheel-center offset as an
-                 adjustable estimate; y_pos denotes the tire center. -->
             <origin xyz="${x_pos} ${y_pos - side_reflect * steering_axis_offset} ${z_pos}" rpy="0.0 0.0 0.0"/>
             <xacro:if value="${is_steer}">
@@ -15,9 +13,4 @@
         </joint>
         <link name="${prefix}_steer_link">
-            <inertial>
-                <origin xyz="0.0 0.0 0.0" rpy="0.0 0.0 0.0"/>
-                <mass value="0.05"/>
-                <inertia ixx="0.0001" ixy="0.0" ixz="0.0" iyy="0.0001" iyz="0.0" izz="0.0001"/>
-            </inertial>
             <visual>
                 <origin xyz="0.0 0.0 0.0" rpy="${-side_reflect * pi/2} 0.0 0.0"/>
@@ -25,7 +18,5 @@
                     <cylinder radius="0.005" length="0.0369"/>
                 </geometry>
-                <material name="green_material">
-                    <color rgba="0.0 1.0 0.0 1.0"/>
-                </material>
+                <material name="steering_material"/>
             </visual>
             <collision>
@@ -44,9 +35,4 @@
         </joint>
         <link name="${prefix}_wheel">
-            <inertial>
-                <origin xyz="0.0 0.0 0.0" rpy="0.0 0.0 0.0"/>
-                <mass value="0.05"/>  <!-- thay vì 0.01 -->
-                <inertia ixx="0.0003" ixy="0.0" ixz="0.0" iyy="0.0003" iyz="0.0" izz="0.0003"/>
-            </inertial>
             <visual>
                 <origin xyz="0.0 0.0 0.0" rpy="0.0 0.0 0.0"/>
@@ -54,7 +40,12 @@
                     <cylinder radius="${wheel_radius}" length="${wheel_width}"/>
                 </geometry>
-                <material name="red_material">
-                    <color rgba="1.0 0.0 0.0 1.0"/>
-                </material>
+                <material name="${'front_wheel_material' if prefix.startswith('front') else 'rear_wheel_material'}"/>
+            </visual>
+            <!-- Estimated outer bevel band: 4.7 mm per side matches the
+                 measured total width while keeping the 40.8 mm tire body. -->
+            <visual>
+                <origin xyz="0.0 0.0 ${side_reflect * (wheel_width / 2.0 + wheel_outer_overhang / 2.0)}"/>
+                <geometry><cylinder radius="${wheel_radius}" length="${wheel_outer_overhang}"/></geometry>
+                <material name="${'front_wheel_material' if prefix.startswith('front') else 'rear_wheel_material'}"/>
             </visual>
             <collision>
@@ -64,4 +55,8 @@
                 </geometry>
             </collision>
+            <collision>
+                <origin xyz="0.0 0.0 ${side_reflect * (wheel_width / 2.0 + wheel_outer_overhang / 2.0)}"/>
+                <geometry><cylinder radius="${wheel_radius}" length="${wheel_outer_overhang}"/></geometry>
+            </collision>
         </link>
     </xacro:macro>
